File: Trail-Traffic-Counter-Board-v10.sch (EAGLE design)
At the start: 45 parts

Commit message: Latest Design
Parts:
- removed MIC5205: (no value), SparkFun-PowerIC:MIC52053.3V
- removed S1: (no value), SparkFun-Electromechanical:SWITCH-SPDTPTH
- added C12: 10uF, SparkFun-Passives:CAP0805
- added C13: 1uF, SparkFun-Capacitors:CAP0805
- added D1: (no value), adafruit:DIODESOD-523
- added NPN: MMBT2222A, SparkFun-DiscreteSemi:TRANSISTOR_NPNMMBT2222A
- added POWER: (no value), SparkFun-Electromechanical:SWITCH-SPDTPTH
- added R13: 100k, SparkFun-Passives:RESISTOR0805-RES
- added R14: 4.7k, SparkFun-Resistors:RESISTOR0805-RES
- added R15, R17: 100, SparkFun-Passives:RESISTOR0805-RES
- added R16: 1k, SparkFun-Passives:RESISTOR0805-RES
- added TC1015: (no value), SparkFun-PowerIC:MIC52053.3V
- added TRIGGER: SN74LVC1G17DBVRG4, Texas Instruments_By_element14_Batch_1:SN74LVC1G17DBVRG4
- renumbered $1_29_$_2016-08-26_17-19-35 to BATT-I2C, JP4 to FTDI-SIMBLEE, JP5 to FTDI-ARDUINO
Connections:
- removed net A2: ATMEGA328P.PC2(ADC2)
- removed net A7: ATMEGA328P.ADC7
- new net HEARTBEAT: ATMEGA328P.ADC7, R14.1, SIMBLEE.P0.04/AIN5
- new net N$14: R15.2, TRIGGER.Y
- new net N$15: NPN.B, R16.1
- new net N$16: NPN.C, R17.2
- new net N$6: C13.2, D1.A, R13.1, R17.1, TRIGGER.A
- new net PWR-DWN: R16.2, SIMBLEE.P0.06/AREF1/AIN7
- new net VIN: C1.1, D1.C, POWER.S, R13.2, TC1015.IN, TRIGGER.VCC
- net !RESET: now also ATMEGA328P.PC2(ADC2)
- net ENABLE: now also R15.1, TC1015.EN; no longer MIC5205.EN, S1.P
- net GND: now also C12.2, C13.1, NPN.E, TC1015.GND, TRIGGER.GND; no longer MIC5205.GND, S1.S
- net N$2: now also TC1015.BP; no longer MIC5205.BP
- net VCC: now also C12.1, R14.2, TC1015.OUT; no longer MIC5205.OUT
- net VRAW: now also POWER.P; no longer C1.1, MIC5205.IN, S1.O
Other:
- note added: "Input: 2.5 to 16V Output 3.3V @ 100mA"
- note added: "N.C."
- note added: "PWR-DWN - Active High Enable - Active High"
- note added: "Provides a 100mSec delay on starup and the ability for the Simblee to reset the board by turning off power."
- note removed: "Input: 2.5 to 16V Output 3.3V @ 150mA"
- note removed: "Optional Pullups for I2C lines"
